File: hardware/MPL3115A2_breakout.brd (EAGLE design)
At the start: 15.2 x 17.8 mm, 16 parts, among them U1 MPL3115A2LGA8

Commit message: Computer change
Parts:
- removed JP5: LOGO-SFESK, SparkFun:SFE-LOGO-FLAME
- removed R1, R2: 1k, SparkFun:0402-RES
- added R3, R4: 4.7K, SparkFun-Resistors:0603-RES
- C1, C3, C4: device SparkFun:0402-CAP -> SparkFun-Capacitors:0603-CAP
- C2: device SparkFun:EIA3216 -> SparkFun-Capacitors:EIA3216
- moved JP1 7.58 mm to (4.32, 10.8), flipped to the top, turned to 90 degrees
- moved C4 0.86 mm to (10.4, 9.71)
- moved C1 0.85 mm to (8.67, 9.71)
- moved C3 0.79 mm to (7.00, 8.41)
Connections:
- net SCL: now also R3.1; no longer R1.1
- net SDA: now also R4.1; no longer R2.1
- net VCC: now also R3.2, R4.2; no longer R1.2, R2.2
Routing:
- net SCL: track 13.3 -> 16.5 mm
- net VCC: track 32.9 -> 35.7 mm
- net SDA: track 14.6 -> 16.2 mm
- net INT1: track 14.9 -> 16.5 mm
- net N$3: track 4.70 -> 5.40 mm
